File: DIMM_Connector_sch.kicad_sch (KiCad schematic)
At the start: 1 part

Commit message: Update schametic 1. Adding 7 DRAMS, 2. Replacing a SPD EEPROM with new one that is including in a temperature sensor, 3. modifying a DIMM Connector and DRAM PAD
Connections:
- net ADDR_BA1: no longer U2.62 (ACT_n)
- net DQ16: now also U2.27 (DQ16); no longer U2.527 (DQ16)
- net SPD_SA2: now reaches U2.238 (SA2)
- net +VTT_0V6 renamed VTT_0V6
- net EXT_12V renamed EXT_1V2
- net VREFCA_2V5 renamed VREFCA_0V6
- new net ACT_n: U2.62 (ACT_n)
- no-connect marks 44 -> 43
Changed lines of the file:
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@@
 	)
 	(junction
-		(at 67.31 19.05)
-		(diameter 0)
-		(color 0 0 0 0)
-	)
-	(junction
 		(at 67.31 115.57)
 		(diameter 0)
@@
 	)
 	(junction
+		(at 67.31 19.05)
+		(diameter 0)
+		(color 0 0 0 0)
+	)
+	(junction
 		(at 92.71 107.95)
 		(diameter 0)
@@
 	)
 	(no_connect
-		(at 227.33 58.42)
-	)
-	(no_connect
 		(at 243.84 138.43)
 	)
@@
 	(wire
 		(pts
+			(xy 226.06 58.42) (xy 227.33 58.42)
+		)
+		(stroke
+			(width 0)
+			(type default)
+		)
+	)
+	(wire
+		(pts
 			(xy 67.31 115.57) (xy 67.31 118.11)
 		)
@@
 	(wire
 		(pts
+			(xy 63.5 19.05) (xy 67.31 19.05)
+		)
+		(stroke
+			(width 0)
+			(type default)
+		)
+	)
+	(wire
+		(pts
 			(xy 67.31 26.67) (xy 67.31 29.21)
 		)
@@
 	(wire
 		(pts
+			(xy 63.5 21.59) (xy 63.5 19.05)
+		)
+		(stroke
+			(width 0)
+			(type default)
+		)
+	)
+	(wire
+		(pts
 			(xy 92.71 135.89) (xy 92.71 133.35)
 		)
@@
 	(wire
 		(pts
-			(xy 59.69 19.05) (xy 67.31 19.05)
-		)
-		(stroke
-			(width 0)
-			(type default)
-		)
-	)
-	(wire
-		(pts
 			(xy 92.71 123.19) (xy 92.71 120.65)
 		)
@@
 		)
 	)
-	(global_label "ADDR_BA1"
+	(global_label "ACT_n"
 		(shape bidirectional)
 		(at 176.53 99.06 180)
@@
 		)
 		(property "Intersheetrefs" "${INTERSHEET_REFS}"
-			(at 162.9992 99.06 0)
+			(at 166.9907 99.06 0)
 			(hide yes)
 			(show_name no)
@@
 		)
 	)
+	(global_label "SPD_SA2"
+		(shape bidirectional)
+		(at 226.06 58.42 180)
+		(fields_autoplaced yes)
+		(effects
+			(font
+				(size 1.27 1.27)
+			)
+			(justify right)
+		)
+		(property "Intersheetrefs" "${INTERSHEET_REFS}"
+			(at 213.7388 58.42 0)
+			(hide yes)
+			(show_name no)
+			(do_not_autoplace no)
+			(effects
+				(font
+					(size 1.27 1.27)
+				)
+				(justify right)
+			)
+		)
+	)
 	(global_label "DQ39"
 		(shape bidirectional)
@@
 			)
 		)
-		(property "Value" "+VTT_0V6"
+		(property "Value" "VTT_0V6"
 			(at 25.908 114.3 0)
 			(show_name no)
@@
 			)
 		)
-		(property "Value" "VREFCA_2V5"
+		(property "Value" "VREFCA_0V6"
 			(at 46.99 147.574 0)
 			(show_name no)
@@
 			)
 		)
-		(property "Value" "EXT_12V"
+		(property "Value" "EXT_1V2"
 			(at 26.67 15.24 0)
 			(show_name no)
@@
 	)
 	(symbol
-		(lib_id "power:GNDREF")
-		(at 59.69 19.05 0)
-		(unit 1)
-		(body_style 1)
-		(exclude_from_sim no)
-		(in_bom yes)
-		(on_board yes)
-		(in_pos_files yes)
-		(dnp no)
-		(fields_autoplaced yes)
-		(property "Reference" "#PWR01"
-			(at 59.69 25.4 0)
-			(hide yes)
-			(show_name no)
-			(do_not_autoplace no)
-			(effects
-				(font
-					(size 1.27 1.27)
-				)
-			)
-		)
-		(property "Value" "GND"
-			(at 59.69 24.13 0)
-			(hide yes)
-			(show_name no)
-			(do_not_autoplace no)
-			(effects
-				(font
-					(size 1.27 1.27)
-				)
-			)
-		)
-		(property "Footprint" ""
-			(at 59.69 19.05 0)
-			(hide yes)
-			(show_name no)
-			(do_not_autoplace no)
-			(effects
-				(font
-					(size 1.27 1.27)
-				)
-			)
-		)
-		(property "Datasheet" ""
-			(at 59.69 19.05 0)
-			(hide yes)
-			(show_name no)
-			(do_not_autoplace no)
-			(effects
-				(font
-					(size 1.27 1.27)
-				)
-			)
-		)
-		(property "Description" "Power symbol creates a global label with name \"GNDREF\" , reference supply ground"
-			(at 59.69 19.05 0)
-			(hide yes)
-			(show_name no)
-			(do_not_autoplace no)
-			(effects
-				(font
-					(size 1.27 1.27)
-				)
-			)
-		)
-		(pin "1"
-		)
-		(instances
-			(project "DDR4_DIMM"
-				(path "/2162f80d-5bbc-406a-8824-9611d78b7103/6efc1bd6-04be-4131-af6a-de12b5fe06f0"
-					(reference "#PWR01")
-					(unit 1)
-				)
-			)
-		)
-	)
-	(symbol
 		(lib_id "DDR4_DRAM_DIMM:DIMM_Connector_288Pin")
 		(at 229.87 93.98 0)
@@
 	)
 	(symbol
+		(lib_name "DIMM_Connector_288Pin_1")
 		(lib_id "DDR4_DRAM_DIMM:DIMM_Connector_288Pin")
 		(at 129.54 20.32 0)
@@
 		(pin "4"
 		)
-		(pin "527"
+		(pin "27"
 		)
 		(pin "196"
@@
 				)
 			)
+		)
+	)
+	(symbol
+		(lib_id "power:GND")
+		(at 63.5 21.59 0)
+		(unit 1)
+		(body_style 1)
+		(exclude_from_sim no)
+		(in_bom yes)
+		(on_board yes)
+		(in_pos_files yes)
+		(dnp no)
+		(fields_autoplaced yes)
+		(property "Reference" "#PWR01"
+			(at 63.5 27.94 0)
+			(hide yes)
+			(show_name no)
+			(do_not_autoplace no)
+			(effects
+				(font
+					(size 1.27 1.27)
+				)
+			)
+		)
+		(property "Value" "GND"
+			(at 63.5 26.67 0)
+			(show_name no)
+			(do_not_autoplace no)
+			(effects
+				(font
+					(size 1.27 1.27)
+				)
+			)
+		)
+		(property "Footprint" ""
+			(at 63.5 21.59 0)
+			(hide yes)
+			(show_name no)
+			(do_not_autoplace no)
+			(effects
+				(font
+					(size 1.27 1.27)
+				)
+			)
+		)
+		(property "Datasheet" ""
+			(at 63.5 21.59 0)
+			(hide yes)
+			(show_name no)
+			(do_not_autoplace no)
+			(effects
+				(font
+					(size 1.27 1.27)
+				)
+			)
+		)
+		(property "Description" "Power symbol creates a global label with name \"GND\" , ground"
+			(at 63.5 21.59 0)
+			(hide yes)
+			(show_name no)
+			(do_not_autoplace no)
+			(effects
+				(font
+					(size 1.27 1.27)
+				)
+			)
+		)
+		(pin "1"
+		)
+		(instances
+			(project "DDR4_DIMM"
+				(path "/2162f80d-5bbc-406a-8824-9611d78b7103/6efc1bd6-04be-4131-af6a-de12b5fe06f0"
+					(reference "#PWR01")
+					(unit 1)
+				)
+			)

Commit message: Modifying stack up from 8 layers to 6 layers and DRAM 5-8 Schematic restore.
Parts:
- renumbered U2 to U1
Changed lines of the file:
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@@
 		(dnp no)
 		(fields_autoplaced yes)
-		(property "Reference" "U2"
+		(property "Reference" "U1"
 			(at 80.518 13.97 0)
 			(show_name no)
@@
 			(project "DDR4_DIMM"
 				(path "/2162f80d-5bbc-406a-8824-9611d78b7103/6efc1bd6-04be-4131-af6a-de12b5fe06f0"
-					(reference "U2")
+					(reference "U1")
 					(unit 18)
 				)
@@
 		(in_pos_files yes)
 		(dnp no)
-		(property "Reference" "#PWR04"
+		(property "Reference" "#PWR03"
 			(at 26.67 121.92 0)
 			(hide yes)
@@
 			(project "DDR4_DIMM"
 				(path "/2162f80d-5bbc-406a-8824-9611d78b7103/6efc1bd6-04be-4131-af6a-de12b5fe06f0"
-					(reference "#PWR04")
+					(reference "#PWR03")
 					(unit 1)
 				)
@@
 		(in_pos_files yes)
 		(dnp no)
-		(property "Reference" "#PWR06"
+		(property "Reference" "#PWR05"
 			(at 46.99 154.94 0)
 			(hide yes)
@@
 			(project "DDR4_DIMM"
 				(path "/2162f80d-5bbc-406a-8824-9611d78b7103/6efc1bd6-04be-4131-af6a-de12b5fe06f0"
-					(reference "#PWR06")
+					(reference "#PWR05")
 					(unit 1)
 				)
@@
 		(dnp no)
 		(fields_autoplaced yes)
-		(property "Reference" "U2"
+		(property "Reference" "U1"
 			(at 138.43 131.9557 0)
 			(show_name no)
@@
 			(project "DDR4_DIMM"
 				(path "/2162f80d-5bbc-406a-8824-9611d78b7103/6efc1bd6-04be-4131-af6a-de12b5fe06f0"
-					(reference "U2")
+					(reference "U1")
 					(unit 12)
 				)
@@
 		(in_pos_files yes)
 		(dnp no)
-		(property "Reference" "U2"
+		(property "Reference" "U1"
 			(at 51.816 119.38 0)
 			(show_name no)
@@
 			(project "DDR4_DIMM"
 				(path "/2162f80d-5bbc-406a-8824-9611d78b7103/6efc1bd6-04be-4131-af6a-de12b5fe06f0"
-					(reference "U2")
+					(reference "U1")
 					(unit 20)
 				)
@@
 		(dnp no)
 		(fields_autoplaced yes)
-		(property "Reference" "U2"
+		(property "Reference" "U1"
 			(at 200.66 77.3457 0)
 			(show_name no)
@@
 			(project "DDR4_DIMM"
 				(path "/2162f80d-5bbc-406a-8824-9611d78b7103/6efc1bd6-04be-4131-af6a-de12b5fe06f0"
-					(reference "U2")
+					(reference "U1")
 					(unit 4)
 				)
@@
 		(dnp no)
 		(fields_autoplaced yes)
-		(property "Reference" "U2"
+		(property "Reference" "U1"
 			(at 52.07 52.0727 0)
 			(show_name no)
@@
 			(project "DDR4_DIMM"
 				(path "/2162f80d-5bbc-406a-8824-9611d78b7103/6efc1bd6-04be-4131-af6a-de12b5fe06f0"
-					(reference "U2")
+					(reference "U1")
 					(unit 9)
 				)
@@
 		(dnp no)
 		(fields_autoplaced yes)
-		(property "Reference" "U2"
+		(property "Reference" "U1"
 			(at 199.39 88.9027 0)
 			(show_name no)
@@
 			(project "DDR4_DIMM"
 				(path "/2162f80d-5bbc-406a-8824-9611d78b7103/6efc1bd6-04be-4131-af6a-de12b5fe06f0"
-					(reference "U2")
+					(reference "U1")
 					(unit 5)
 				)
@@
 		(in_pos_files yes)
 		(dnp no)
-		(property "Reference" "#PWR02"
+		(property "Reference" "#PWR01"
 			(at 26.67 22.86 0)
 			(hide yes)
@@
 			(project "DDR4_DIMM"
 				(path "/2162f80d-5bbc-406a-8824-9611d78b7103/6efc1bd6-04be-4131-af6a-de12b5fe06f0"
-					(reference "#PWR02")
+					(reference "#PWR01")
 					(unit 1)
 				)
@@
 		(dnp no)
 		(fields_autoplaced yes)
-		(property "Reference" "U2"
+		(property "Reference" "U1"
 			(at 199.39 139.5757 0)
 			(show_name no)
@@
 			(project "DDR4_DIMM"
 				(path "/2162f80d-5bbc-406a-8824-9611d78b7103/6efc1bd6-04be-4131-af6a-de12b5fe06f0"
-					(reference "U2")
+					(reference "U1")
 					(unit 19)
 				)
@@
 		(dnp no)
 		(fields_autoplaced yes)
-		(property "Reference" "U2"
+		(property "Reference" "U1"
 			(at 201.93 44.5797 0)
 			(show_name no)
@@
 			(project "DDR4_DIMM"
 				(path "/2162f80d-5bbc-406a-8824-9611d78b7103/6efc1bd6-04be-4131-af6a-de12b5fe06f0"
-					(reference "U2")
+					(reference "U1")
 					(unit 2)
 				)
@@
 		(dnp no)
 		(fields_autoplaced yes)
-		(property "Reference" "U2"
+		(property "Reference" "U1"
 			(at 138.43 168.7857 0)
 			(show_name no)
@@
 			(project "DDR4_DIMM"
 				(path "/2162f80d-5bbc-406a-8824-9611d78b7103/6efc1bd6-04be-4131-af6a-de12b5fe06f0"
-					(reference "U2")
+					(reference "U1")
 					(unit 7)
 				)
@@
 		(in_pos_files yes)
 		(dnp no)
-		(property "Reference" "#PWR03"
+		(property "Reference" "#PWR02"
 			(at 26.67 99.06 0)
 			(hide yes)
@@
 			(project "DDR4_DIMM"
 				(path "/2162f80d-5bbc-406a-8824-9611d78b7103/6efc1bd6-04be-4131-af6a-de12b5fe06f0"
-					(reference "#PWR03")
+					(reference "#PWR02")
 					(unit 1)
 				)
@@
 		(dnp no)
 		(fields_autoplaced yes)
-		(property "Reference" "U2"
+		(property "Reference" "U1"
 			(at 238.76 97.6657 0)
 			(show_name no)
@@
 			(project "DDR4_DIMM"
 				(path "/2162f80d-5bbc-406a-8824-9611d78b7103/6efc1bd6-04be-4131-af6a-de12b5fe06f0"
-					(reference "U2")
+					(reference "U1")
 					(unit 15)
 				)
@@
 		(dnp no)
 		(fields_autoplaced yes)
-		(property "Reference" "U2"
+		(property "Reference" "U1"
 			(at 129.54 15.24 0)
 			(show_name no)
@@
 			(project "DDR4_DIMM"
 				(path "/2162f80d-5bbc-406a-8824-9611d78b7103/6efc1bd6-04be-4131-af6a-de12b5fe06f0"
-					(reference "U2")
+					(reference "U1")
 					(unit 11)
 				)
@@
 		(dnp no)
 		(fields_autoplaced yes)
-		(property "Reference" "U2"
+		(property "Reference" "U1"
 			(at 248.92 36.9597 0)
 			(show_name no)
@@
 			(project "DDR4_DIMM"
 				(path "/2162f80d-5bbc-406a-8824-9611d78b7103/6efc1bd6-04be-4131-af6a-de12b5fe06f0"
-					(reference "U2")
+					(reference "U1")
 					(unit 17)
 				)
@@
 		(dnp no)
 		(fields_autoplaced yes)
-		(property "Reference" "U2"
+		(property "Reference" "U1"
 			(at 52.07 135.8927 0)
 			(show_name no)
@@
 			(project "DDR4_DIMM"
 				(path "/2162f80d-5bbc-406a-8824-9611d78b7103/6efc1bd6-04be-4131-af6a-de12b5fe06f0"
-					(reference "U2")
+					(reference "U1")
 					(unit 22)
 				)
@@
 		(in_pos_files yes)
 		(dnp no)
-		(property "Reference" "U2"
+		(property "Reference" "U1"
 			(at 50.546 100.076 0)
 			(show_name no)
@@
 			(project "DDR4_DIMM"
 				(path "/2162f80d-5bbc-406a-8824-9611d78b7103/6efc1bd6-04be-4131-af6a-de12b5fe06f0"
-					(reference "U2")
+					(reference "U1")
 					(unit 13)
 				)
@@
 		(dnp no)
 		(fields_autoplaced yes)
-		(property "Reference" "U2"
+		(property "Reference" "U1"
 			(at 60.96 146.05 0)
 			(show_name no)
@@
 			(project "DDR4_DIMM"
 				(path "/2162f80d-5bbc-406a-8824-9611d78b7103/6efc1bd6-04be-4131-af6a-de12b5fe06f0"
-					(reference "U2")
+					(reference "U1")
 					(unit 8)
 				)
@@
 		(dnp no)
 		(fields_autoplaced yes)
-		(property "Reference" "U2"
+		(property "Reference" "U1"
 			(at 238.76 137.2897 0)
 			(show_name no)
@@
 			(project "DDR4_DIMM"
 				(path "/2162f80d-5bbc-406a-8824-9611d78b7103/6efc1bd6-04be-4131-af6a-de12b5fe06f0"
-					(reference "U2")
+					(reference "U1")
 					(unit 14)
 				)
@@
 		(dnp no)
 		(fields_autoplaced yes)
-		(property "Reference" "#PWR01"
+		(property "Reference" "#PWR06"
 			(at 63.5 27.94 0)
 			(hide yes)
@@
 			(project "DDR4_DIMM"
 				(path "/2162f80d-5bbc-406a-8824-9611d78b7103/6efc1bd6-04be-4131-af6a-de12b5fe06f0"
-					(reference "#PWR01")
+					(reference "#PWR06")
 					(unit 1)
 				)
@@
 		(dnp no)
 		(fields_autoplaced yes)
-		(property "Reference" "U2"
+		(property "Reference" "U1"
 			(at 270.51 102.7457 0)
 			(show_name no)
@@
 			(project "DDR4_DIMM"
 				(path "/2162f80d-5bbc-406a-8824-9611d78b7103/6efc1bd6-04be-4131-af6a-de12b5fe06f0"
-					(reference "U2")
+					(reference "U1")
 					(unit 23)
 				)
@@
 		(dnp no)
 		(fields_autoplaced yes)
-		(property "Reference" "U2"
+		(property "Reference" "U1"
 			(at 248.92 77.4727 0)
 			(show_name no)
@@
 			(project "DDR4_DIMM"
 				(path "/2162f80d-5bbc-406a-8824-9611d78b7103/6efc1bd6-04be-4131-af6a-de12b5fe06f0"
-					(reference "U2")
+					(reference "U1")
 					(unit 6)
 				)
@@
 		(dnp no)
 		(fields_autoplaced yes)
-		(property "Reference" "U2"
+		(property "Reference" "U1"
 			(at 199.39 100.7137 0)
 			(show_name no)
@@
 			(project "DDR4_DIMM"
 				(path "/2162f80d-5bbc-406a-8824-9611d78b7103/6efc1bd6-04be-4131-af6a-de12b5fe06f0"
-					(reference "U2")
+					(reference "U1")
 					(unit 1)
 				)
@@
 		(dnp no)
 		(fields_autoplaced yes)
-		(property "Reference" "U2"
+		(property "Reference" "U1"
 			(at 199.39 118.3667 0)
 			(show_name no)
@@
 			(project "DDR4_DIMM"
 				(path "/2162f80d-5bbc-406a-8824-9611d78b7103/6efc1bd6-04be-4131-af6a-de12b5fe06f0"
-					(reference "U2")
+					(reference "U1")
 					(unit 3)
 				)
@@
 		(dnp no)
 		(fields_autoplaced yes)
-		(property "Reference" "U2"
+		(property "Reference" "U1"
 			(at 248.92 55.7557 0)
 			(show_name no)
@@
 			(project "DDR4_DIMM"
 				(path "/2162f80d-5bbc-406a-8824-9611d78b7103/6efc1bd6-04be-4131-af6a-de12b5fe06f0"
-					(reference "U2")
+					(reference "U1")
 					(unit 21)
 				)
@@
 		(in_pos_files yes)
 		(dnp no)
-		(property "Reference" "U2"
+		(property "Reference" "U1"
 			(at 248.92 24.892 0)
 			(show_name no)
@@
 			(project "DDR4_DIMM"
 				(path "/2162f80d-5bbc-406a-8824-9611d78b7103/6efc1bd6-04be-4131-af6a-de12b5fe06f0"
-					(reference "U2")
+					(reference "U1")
 					(unit 16)
 				)
@@
 		(dnp no)
 		(fields_autoplaced yes)
-		(property "Reference" "U2"
+		(property "Reference" "U1"
 			(at 270.51 139.5757 0)
 			(show_name no)
@@
 			(project "DDR4_DIMM"
 				(path "/2162f80d-5bbc-406a-8824-9611d78b7103/6efc1bd6-04be-4131-af6a-de12b5fe06f0"
-					(reference "U2")
+					(reference "U1")
 					(unit 10)
 				)
@@
 		(in_pos_files yes)
 		(dnp no)
-		(property "Reference" "#PWR05"
+		(property "Reference" "#PWR04"
 			(at 27.94 138.43 0)
 			(hide yes)
@@
 			(project "DDR4_DIMM"
 				(path "/2162f80d-5bbc-406a-8824-9611d78b7103/6efc1bd6-04be-4131-af6a-de12b5fe06f0"
-					(reference "#PWR05")
+					(reference "#PWR04")
 					(unit 1)
 				)
