File: DRAM_5to8.kicad_sch (KiCad schematic)
At the start: 88 parts, among them U2 K4A8G085WC-BCPB, U3 K4A8G085WC-BCPB, U4 K4A8G085WC-BCPB, U5 K4A8G085WC-BCPB

Commit message: Modifying stack up from 8 layers to 6 layers and DRAM 5-8 Schematic restore.
Parts:
- removed C1, C11, C18, C19, C23, C30, C31, C35, C38, C39, C8, C9: 1uF, DDR4_DRAM_DIMM:C_0402_1005, symbol Mixed_signal:CAP_1608
- removed C10, C12, C17, C2, C20, C26, C27, C34, C36, C37, C40, C7: 0.1uF, DDR4_DRAM_DIMM:C_0402_1005, symbol Mixed_signal:CAP_1608
- removed C13, C14, C21, C22, C28, C29, C3, C4: 1uF, DDR4_DRAM_DIMM:C_0402_1005, symbol Mixed_signal:CAP_1005
- removed C15, C16, C24, C25, C32, C33, C5, C6: 100nF, DDR4_DRAM_DIMM:C_0402_1005, symbol Mixed_signal:CAP_1005
- removed L1, L2, L3, L4, L5, L6, L7, L8: MPZ1608S221A, DDR4_DRAM_DIMM:MPZ1608S260ATAH0, symbol MPZ1608S260ATAH0:MPZ1608S221A
- removed R1, R10, R11, R12, R13, R14, R15, R16, R17, R19, R2, R20, R21, R22, R23, R24, R25, R26, R28, R29, R3, R30, R31, R32, R33, R34, R35, R4, R5, R6, R7, R8: 15, DDR4_DRAM_DIMM:R_0402_1005, symbol Mixed_signal:RES_1005
- removed R18, R27, R36, R9: 240/1%, DDR4_DRAM_DIMM:R_0402_1005, symbol Mixed_signal:RES_1005
- removed U2: K4A8G085WC-BCPB, K4A8G085WC-BCPB, symbol DDR4_DIMM:K4A8G085WC-BCPB
- removed U3, U4, U5: K4A8G085WC-BCPB, DDR4_DRAM_DIMM:K4A8G085WC-BCPB, symbol DDR4_DIMM:K4A8G085WC-BCPB
- added C41, C48, C49, C51, C58, C59, C63, C70, C71, C75, C78, C79: 1uF, DDR4_DRAM_DIMM:C_0402_1005, symbol Mixed_signal:CAP_1608
- added C42, C47, C50, C52, C57, C60, C66, C67, C74, C76, C77, C80: 0.1uF, DDR4_DRAM_DIMM:C_0402_1005, symbol Mixed_signal:CAP_1608
- added C43, C44, C53, C54, C61, C62, C68, C69: 1uF, DDR4_DRAM_DIMM:C_0402_1005, symbol Mixed_signal:CAP_1005
- added C45, C46, C55, C56, C64, C65, C72, C73: 100nF, DDR4_DRAM_DIMM:C_0402_1005, symbol Mixed_signal:CAP_1005
- added L10, L11, L12, L13, L14, L15, L16, L9: MPZ1608S221A, DDR4_DRAM_DIMM:MPZ1608S260ATAH0, symbol MPZ1608S260ATAH0:MPZ1608S221A
- added R37, R38, R39, R40, R41, R42, R43, R44, R46, R47, R48, R49, R50, R51, R52, R53, R55, R56, R57, R58, R59, R60, R61, R62, R64, R65, R66, R67, R68, R69, R70, R71: 15, DDR4_DRAM_DIMM:R_0402_1005, symbol Mixed_signal:RES_1005
- added R45, R54, R63, R72: 240/1%, DDR4_DRAM_DIMM:R_0402_1005, symbol Mixed_signal:RES_1005
- added U6: K4A8G085WC-BCPB, K4A8G085WC-BCPB, symbol DDR4_DIMM:K4A8G085WC-BCPB
- added U7, U8, U9: K4A8G085WC-BCPB, DDR4_DRAM_DIMM:K4A8G085WC-BCPB, symbol DDR4_DIMM:K4A8G085WC-BCPB
Connections:
- net ACT_n: now also U6.H3 (ACT_n), U7.H3 (ACT_n), U8.H3 (ACT_n), U9.H3 (ACT_n)
- net ADDR_A0: now also U6.L3 (A0), U7.L3 (A0), U8.L3 (A0), U9.L3 (A0)
- net ADDR_A1: now also U6.L7 (A1), U7.L7 (A1), U8.L7 (A1), U9.L7 (A1)
- net ADDR_A10: now also U6.J3 (A10/AP), U7.J3 (A10/AP), U8.J3 (A10/AP), U9.J3 (A10/AP)
- net ADDR_A11: now also U6.N2 (A11), U7.N2 (A11), U8.N2 (A11), U9.N2 (A11)
- net ADDR_A12: now also U6.J7 (A12/BC_n), U7.J7 (A12/BC_n), U8.J7 (A12/BC_n), U9.J7 (A12/BC_n)
- net ADDR_A13: now also U6.N8 (A13), U7.N8 (A13), U8.N8 (A13), U9.N8 (A13)
- net ADDR_A14: now also U6.H2 (WE_n/A14), U7.H2 (WE_n/A14), U8.H2 (WE_n/A14), U9.H2 (WE_n/A14)
- net ADDR_A15: now also U6.H7 (CAS_n/A15), U7.H7 (CAS_n/A15), U8.H7 (CAS_n/A15), U9.H7 (CAS_n/A15)
- net ADDR_A16: now also U6.H8 (RAS_n), U7.H8 (RAS_n), U8.H8 (RAS_n), U9.H8 (RAS_n)
- net ADDR_A2: now also U6.M3 (A2), U7.M3 (A2), U8.M3 (A2), U9.M3 (A2)
- net ADDR_A3: now also U6.K7 (A3), U7.K7 (A3), U8.K7 (A3), U9.K7 (A3)
- net ADDR_A4: now also U6.K3 (A4), U7.K3 (A4), U8.K3 (A4), U9.K3 (A4)
- net ADDR_A5: now also U6.L8 (A5), U7.L8 (A5), U8.L8 (A5), U9.L8 (A5)
- net ADDR_A6: now also U6.L2 (A6), U7.L2 (A6), U8.L2 (A6), U9.L2 (A6)
- net ADDR_A7: now also U6.M8 (A7), U7.M8 (A7), U8.M8 (A7), U9.M8 (A7)
- net ADDR_A8: now also U6.M2 (A8), U7.M2 (A8), U8.M2 (A8), U9.M2 (A8)
- net ADDR_A9: now also U6.M7 (A9), U7.M7 (A9), U8.M7 (A9), U9.M7 (A9)
- net ADDR_BA0: now also U6.K2 (BA0), U7.K2 (BA0), U8.K2 (BA0), U9.K2 (BA0)
- net ADDR_BA1: now also U6.K8 (BA1), U7.K8 (BA1), U8.K8 (BA1), U9.K8 (BA1)
- net ADDR_BG0: now also U6.J2 (BG0), U7.J2 (BG0), U8.J2 (BG0), U9.J2 (BG0)
- net ADDR_BG1: now also U6.J8 (BG1), U7.J8 (BG1), U8.J8 (BG1), U9.J8 (BG1)
- net ADDR_CS0: now also U6.G7 (CS_n), U7.G7 (CS_n), U8.G7 (CS_n), U9.G7 (CS_n)
- net CLK0_N: now also U6.F8 (CK_c), U7.F8 (CK_c), U8.F8 (CK_c), U9.F8 (CK_c)
- net CLK0_P: now also U6.F7 (CK_t), U7.F7 (CK_t), U8.F7 (CK_t), U9.F7 (CK_t)
- net DDR4_ALERT: now also U6.L9 (ALERT_n), U7.L9 (ALERT_n), U8.L9 (ALERT_n), U9.L9 (ALERT_n)
- net DDR4_CKE0: now also U6.G3 (CKE), U7.G3 (CKE), U8.G3 (CKE), U9.G3 (CKE)
- net DDR4_ODT: now also U6.F3 (ODT), U7.F3 (ODT), U8.F3 (ODT), U9.F3 (ODT)
- net DDR4_PARITY: now also U6.N3 (PAR), U7.N3 (PAR), U8.N3 (PAR), U9.N3 (PAR)
- net DDR4_RESET: now also U6.L1 (RESET_n), U7.L1 (RESET_n), U8.L1 (RESET_n), U9.L1 (RESET_n)
- net DQ32: now also R37.1
- net DQ33: now also R38.1
- net DQ34: now also R39.1
- net DQ35: now also R40.1
- net DQ36: now also R41.1
- net DQ37: now also R42.1
- net DQ38: now also R43.1
- net DQ39: now also R44.1
- net DQ40: now also R46.1
- net DQ41: now also R47.1
- net DQ42: now also R48.1
- net DQ43: now also R49.1
- net DQ44: now also R50.1
- net DQ45: now also R51.1
- net DQ46: now also R52.1
- net DQ47: now also R53.1
- net DQ48: now also R55.1
- net DQ49: now also R56.1
- net DQ50: now also R57.1
- net DQ51: now also R58.1
- net DQ52: now also R59.1
- net DQ53: now also R60.1
- net DQ54: now also R61.1
- net DQ55: now also R62.1
- net DQ56: now also R64.1
- net DQ57: now also R65.1
- net DQ58: now also R66.1
- net DQ59: now also R67.1
- net DQ60: now also R68.1
- net DQ61: now also R69.1
- net DQ62: now also R70.1
- net DQ63: now also R71.1
- net DQS4_N: now also U6.B3 (DQS_c)
- net DQS4_P: now also U6.C3 (DQS_t)
- net DQS5_N: now also U7.B3 (DQS_c)
- net DQS5_P: now also U7.C3 (DQS_t)
- net DQS6_N: now also U8.B3 (DQS_c)
- net DQS6_P: now also U8.C3 (DQS_t)
- net DQS7_N: now also U9.B3 (DQS_c)
- net DQS7_P: now also U9.C3 (DQS_t)
- net GND: now also C41.1, C42.1, C43.1, C44.1, C45.1, C46.1, C47.1, C48.1, C49.1, C50.1, C51.1, C52.1, C53.1, C54.1, C55.1, C56.1, C57.1, C58.1, C59.1, C60.1, C61.1, C62.1, C63.1, C64.1, C65.1, C66.1, C67.1, C68.1, C69.1, C70.1, C71.1, C72.1, C73.1, C74.1, C75.1, C76.1, C77.1, C78.1, C79.1, C80.1, R45.2, R54.2, R63.2, R72.2, U6.A2 (VSSQ), U6.A8 (VSSQ), U6.A9 (VSS), U6.C8 (VSS), U6.D1 (VSSQ), U6.D9 (VSSQ), U6.E1 (VSS), U6.E9 (VSS), U6.G1 (VSS), U6.H9 (VSS), U6.K1 (VSS), U6.K9 (VSS), U6.N1 (VSS), U7.A2 (VSSQ), U7.A8 (VSSQ), U7.A9 (VSS), U7.C8 (VSS), U7.D1 (VSSQ), U7.D9 (VSSQ), U7.E1 (VSS), U7.E9 (VSS), U7.G1 (VSS), U7.H9 (VSS), U7.K1 (VSS), U7.K9 (VSS), U7.N1 (VSS), U8.A2 (VSSQ), U8.A8 (VSSQ), U8.A9 (VSS), U8.C8 (VSS), U8.D1 (VSSQ), U8.D9 (VSSQ), U8.E1 (VSS), U8.E9 (VSS), U8.G1 (VSS), U8.H9 (VSS), U8.K1 (VSS), U8.K9 (VSS), U8.N1 (VSS), U9.A2 (VSSQ), U9.A8 (VSSQ), U9.A9 (VSS), U9.C8 (VSS), U9.D1 (VSSQ), U9.D9 (VSSQ), U9.E1 (VSS), U9.E9 (VSS), U9.G1 (VSS), U9.H9 (VSS), U9.K1 (VSS), U9.K9 (VSS), U9.N1 (VSS)
- net VDD_1V2: now also L10.2, L11.2, L12.2, L13.2, L14.2, L15.2, L16.2, L9.2
- net VDD_2V5: now also C49.2, C50.2, C59.2, C60.2, C71.2, C74.2, C79.2, C80.2, U6.B1 (VPP), U6.M9 (VPP), U7.B1 (VPP), U7.M9 (VPP), U8.B1 (VPP), U8.M9 (VPP), U9.B1 (VPP), U9.M9 (VPP)
- net VREFCA_0V6: now also U6.J1 (VREFCA), U7.J1 (VREFCA), U8.J1 (VREFCA), U9.J1 (VREFCA)
- new net: R46.2, U7.C2 (DQ0)
- new net: R54.1, U7.B9 (ZQ)
- new net: R67.2, U9.D7 (DQ3)
- new net: R63.1, U8.B9 (ZQ)
- new net: R42.2, U6.D8 (DQ5)
- new net: R65.2, U9.B7 (DQ1)
- new net: R64.2, U9.C2 (DQ0)
- new net: R68.2, U9.D2 (DQ4)
- new net: R66.2, U9.D3 (DQ2)
- new net: R69.2, U9.D8 (DQ5)
- new net: R70.2, U9.E3 (DQ6)
- new net: R71.2, U9.E7 (DQ7)
- new net: R38.2, U6.B7 (DQ1)
- new net: R37.2, U6.C2 (DQ0)
- new net: R41.2, U6.D2 (DQ4)
- new net: R39.2, U6.D3 (DQ2)
- new net: R40.2, U6.D7 (DQ3)
- new net: R43.2, U6.E3 (DQ6)
- new net: R44.2, U6.E7 (DQ7)
- new net: R45.1, U6.B9 (ZQ)
- new net: R51.2, U7.D8 (DQ5)
- new net: R47.2, U7.B7 (DQ1)
- new net: R50.2, U7.D2 (DQ4)
- new net: R48.2, U7.D3 (DQ2)
- new net: R49.2, U7.D7 (DQ3)
- new net: R52.2, U7.E3 (DQ6)
- new net: R53.2, U7.E7 (DQ7)
- new net: R55.2, U8.C2 (DQ0)
- new net: R61.2, U8.E3 (DQ6)
- new net: R62.2, U8.E7 (DQ7)
- new net: R72.1, U9.B9 (ZQ)
- new net: R59.2, U8.D2 (DQ4)
- new net: R58.2, U8.D7 (DQ3)
- new net: R60.2, U8.D8 (DQ5)
- new net: R57.2, U8.D3 (DQ2)
- new net: R56.2, U8.B7 (DQ1)
- new net VDDQ5_1V2: C44.2, C46.2, C47.2, C48.2, L10.1, U6.B2 (VDDQ), U6.B8 (VDDQ), U6.C1 (VDDQ), U6.C9 (VDDQ), U6.E2 (VDDQ), U6.E8 (VDDQ)
- new net VDDQ6_1V2: C54.2, C56.2, C57.2, C58.2, L12.1, U7.B2 (VDDQ), U7.B8 (VDDQ), U7.C1 (VDDQ), U7.C9 (VDDQ), U7.E2 (VDDQ), U7.E8 (VDDQ)
- new net VDDQ7_1V2: C62.2, C65.2, C67.2, C70.2, L14.1, U8.B2 (VDDQ), U8.B8 (VDDQ), U8.C1 (VDDQ), U8.C9 (VDDQ), U8.E2 (VDDQ), U8.E8 (VDDQ)
- new net VDDQ8_1V2: C69.2, C73.2, C77.2, C78.2, L16.1, U9.B2 (VDDQ), U9.B8 (VDDQ), U9.C1 (VDDQ), U9.C9 (VDDQ), U9.E2 (VDDQ), U9.E8 (VDDQ)
- new net VDRAM5_1V2: C41.2, C42.2, C43.2, C45.2, L9.1, U6.A1 (VDD), U6.C7 (VDD), U6.F1 (VDD), U6.F9 (VDD), U6.H1 (VDD), U6.J9 (VDD), U6.M1 (VDD), U6.N9 (VDD)
- new net VDRAM6_1V2: C51.2, C52.2, C53.2, C55.2, L11.1, U7.A1 (VDD), U7.C7 (VDD), U7.F1 (VDD), U7.F9 (VDD), U7.H1 (VDD), U7.J9 (VDD), U7.M1 (VDD), U7.N9 (VDD)
- new net VDRAM7_1V2: C61.2, C63.2, C64.2, C66.2, L13.1, U8.A1 (VDD), U8.C7 (VDD), U8.F1 (VDD), U8.F9 (VDD), U8.H1 (VDD), U8.J9 (VDD), U8.M1 (VDD), U8.N9 (VDD)
- new net VDRAM8_1V2: C68.2, C72.2, C75.2, C76.2, L15.1, U9.A1 (VDD), U9.C7 (VDD), U9.F1 (VDD), U9.F9 (VDD), U9.H1 (VDD), U9.J9 (VDD), U9.M1 (VDD), U9.N9 (VDD)
