File: Power_Magnagement_sch.kicad_sch (KiCad schematic)
At the start: 0 parts

Commit message: Update schametic 1. Adding 7 DRAMS, 2. Replacing a SPD EEPROM with new one that is including in a temperature sensor, 3. modifying a DIMM Connector and DRAM PAD
Parts:
- added C1, C3: 1uF, Capacitor_SMD:C_01005_0402Metric_Pad0.57x0.30mm_HandSolder, symbol Mixed_signal:CAP_1005
- added C10, C11, C12, C8, C9: 10uF, Capacitor_SMD:C_0603_1608Metric_Pad1.08x0.95mm_HandSolder, symbol Mixed_signal:CAP_1608
- added C4, C6: 100nF, Capacitor_SMD:C_01005_0402Metric_Pad0.57x0.30mm_HandSolder, symbol Mixed_signal:CAP_1005
- added C7: 1nF/1005, Capacitor_SMD:C_01005_0402Metric_Pad0.57x0.30mm_HandSolder, symbol Mixed_signal:CAP_1005
- added CR1: SLVU2.8HTG, DDR4_DRAM_DIMM:SLVU2.8HTG, symbol SLVU2.8HTG:SLVU2.8HTG
- added D1: RCLAMP01211ZCFT, RCLAMP01211ZCFT, symbol RCLAMP01211ZCFT:RCLAMP01211ZCFT
- added L1, L2: MPZ1608S221A, DDR4_DRAM_DIMM:MPZ1608S260ATAH0, symbol MPZ1608S260ATAH0:MPZ1608S221A
- added R1, R2, R3: 10K, RES_0603, symbol Mixed_signal:RES_10K-0.1W-1%-0603
- added R4, R5: 10K/1%, RES_0603, symbol Mixed_signal:RES_10K-0.1W-1%-0603
- added U3: TPS51200AQDRCTQ1, DRC0010J, symbol TPS51200AQDRCTQ1:TPS51200AQDRCTQ1
Connections:
- new net: C7.2, R1.2, R2.2, U3.1 (REFIN)
- new net: R4.1, U3.6 (REFOUT)
- new net: R3.1, U3.9 (PGOOD)
- new net EXT_1V2: D1.1, L1.2
- new net EXT_2V5: CR1.1, CR1.2, L2.2
- new net GND: C1.1, C10.1, C11.1, C12.1, C3.1, C4.1, C6.1, C7.1, C8.1, C9.1, CR1.3, D1.2, R2.1, R5.2, U3.11 (PAD), U3.4 (PGND), U3.8 (GND)
- new net VDDQ_1V2: C8.2, C9.2, R1.1, U3.2 (VLDOIN)
- new net VDD_1V2: C1.2, C4.2, L1.1
- new net VDD_2V5: C3.2, C6.2, L2.1, R3.2, U3.10 (VIN), U3.7 (EN)
- new net VREFCA_0V6: R4.2, R5.1
- new net VTT_0V6: C10.2, C11.2, C12.2, U3.3 (VO), U3.5 (VOSNS)
Other:
- note added: "220ohms @100MHz"
- note added: "source 4.5A / sink 5.5A"

Commit message: Modifying stack up from 8 layers to 6 layers and DRAM 5-8 Schematic restore.
Parts:
- C81: renamed from C1; footprint Capacitor_SMD:C_01005_0402Metric_Pad0.57x0.30mm_HandSolder -> DDR4_DRAM_DIMM:C_0402_1005
- C82: renamed from C3; footprint Capacitor_SMD:C_01005_0402Metric_Pad0.57x0.30mm_HandSolder -> DDR4_DRAM_DIMM:C_0402_1005
- C83: renamed from C4; footprint Capacitor_SMD:C_01005_0402Metric_Pad0.57x0.30mm_HandSolder -> DDR4_DRAM_DIMM:C_0402_1005
- C84: renamed from C6; footprint Capacitor_SMD:C_01005_0402Metric_Pad0.57x0.30mm_HandSolder -> DDR4_DRAM_DIMM:C_0402_1005
- C85: renamed from C7; footprint Capacitor_SMD:C_01005_0402Metric_Pad0.57x0.30mm_HandSolder -> DDR4_DRAM_DIMM:C_0402_1005
- C86: renamed from C8; footprint Capacitor_SMD:C_0603_1608Metric_Pad1.08x0.95mm_HandSolder -> DDR4_DRAM_DIMM:C_0603_1608
- C87: renamed from C9; footprint Capacitor_SMD:C_0603_1608Metric_Pad1.08x0.95mm_HandSolder -> DDR4_DRAM_DIMM:C_0603_1608
- C88: renamed from C10; footprint Capacitor_SMD:C_0603_1608Metric_Pad1.08x0.95mm_HandSolder -> DDR4_DRAM_DIMM:C_0603_1608
- C89: renamed from C11; footprint Capacitor_SMD:C_0603_1608Metric_Pad1.08x0.95mm_HandSolder -> DDR4_DRAM_DIMM:C_0603_1608
- C90: renamed from C12; footprint Capacitor_SMD:C_0603_1608Metric_Pad1.08x0.95mm_HandSolder -> DDR4_DRAM_DIMM:C_0603_1608
- D1: footprint RCLAMP01211ZCFT -> DDR4_DRAM_DIMM:RCLAMP01211ZCFT
- R73: renamed from R1; footprint RES_0603 -> DDR4_DRAM_DIMM:R_0402_1005
- R74: renamed from R2; footprint RES_0603 -> DDR4_DRAM_DIMM:R_0402_1005
- R75: renamed from R3; footprint RES_0603 -> DDR4_DRAM_DIMM:R_0402_1005
- R76: renamed from R4; footprint RES_0603 -> DDR4_DRAM_DIMM:R_0603_1608
- R77: renamed from R5; footprint RES_0603 -> DDR4_DRAM_DIMM:R_0603_1608
- U10: renamed from U3; footprint DRC0010J -> DDR4_DRAM_DIMM:DRC0010J
- renumbered L1 to L17, L2 to L18
