File: SPD_EEPROM.kicad_sch (KiCad schematic)
At the start: 4 parts, among them U7 S-34TS04A0B-A8T5U5

Commit message: Modifying stack up from 8 layers to 6 layers and DRAM 5-8 Schematic restore.
Parts:
- C91: renamed from C43; footprint Capacitor_SMD:C_01005_0402Metric_Pad0.57x0.30mm_HandSolder -> DDR4_DRAM_DIMM:R_0402_1005
- C92: renamed from C44; footprint Capacitor_SMD:C_01005_0402Metric_Pad0.57x0.30mm_HandSolder -> DDR4_DRAM_DIMM:R_0402_1005
- renumbered L11 to L19, U7 to U11
Changed lines of the file:
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@@
 		(dnp no)
 		(fields_autoplaced yes)
-		(property "Reference" "L11"
+		(property "Reference" "L19"
 			(at 86.36 80.01 0)
 			(show_name no)
@@
 			(project "DDR4_DIMM"
 				(path "/2162f80d-5bbc-406a-8824-9611d78b7103/cb7293af-232b-4c7f-85bc-3b7b1ae107bd"
-					(reference "L11")
+					(reference "L19")
 					(unit 1)
 				)
@@
 		(dnp no)
 		(fields_autoplaced yes)
-		(property "Reference" "#PWR036"
+		(property "Reference" "#PWR0180"
 			(at 116.84 118.11 0)
 			(hide yes)
@@
 			(project "DDR4_DIMM"
 				(path "/2162f80d-5bbc-406a-8824-9611d78b7103/cb7293af-232b-4c7f-85bc-3b7b1ae107bd"
-					(reference "#PWR036")
+					(reference "#PWR0180")
 					(unit 1)
 				)
@@
 		(in_pos_files yes)
 		(dnp no)
-		(property "Reference" "C44"
+		(property "Reference" "C92"
 			(at 119.38 100.3299 90)
 			(show_name no)
@@
 			)
 		)
-		(property "Footprint" "Capacitor_SMD:C_01005_0402Metric_Pad0.57x0.30mm_HandSolder"
+		(property "Footprint" "DDR4_DRAM_DIMM:R_0402_1005"
 			(at 113.03 100.33 0)
 			(hide yes)
@@
 			(project "DDR4_DIMM"
 				(path "/2162f80d-5bbc-406a-8824-9611d78b7103/cb7293af-232b-4c7f-85bc-3b7b1ae107bd"
-					(reference "C44")
+					(reference "C92")
 					(unit 1)
 				)
@@
 		(in_pos_files yes)
 		(dnp no)
-		(property "Reference" "C43"
+		(property "Reference" "C91"
 			(at 107.95 100.3299 90)
 			(show_name no)
@@
 			)
 		)
-		(property "Footprint" "Capacitor_SMD:C_01005_0402Metric_Pad0.57x0.30mm_HandSolder"
+		(property "Footprint" "DDR4_DRAM_DIMM:R_0402_1005"
 			(at 101.6 100.33 0)
 			(hide yes)
@@
 			(project "DDR4_DIMM"
 				(path "/2162f80d-5bbc-406a-8824-9611d78b7103/cb7293af-232b-4c7f-85bc-3b7b1ae107bd"
-					(reference "C43")
+					(reference "C91")
 					(unit 1)
 				)
@@
 		(in_pos_files yes)
 		(dnp no)
-		(property "Reference" "#PWR034"
+		(property "Reference" "#PWR0178"
 			(at 71.12 85.09 0)
 			(hide yes)
@@
 			(project "DDR4_DIMM"
 				(path "/2162f80d-5bbc-406a-8824-9611d78b7103/cb7293af-232b-4c7f-85bc-3b7b1ae107bd"
-					(reference "#PWR034")
+					(reference "#PWR0178")
 					(unit 1)
 				)
@@
 		(dnp no)
 		(fields_autoplaced yes)
-		(property "Reference" "#PWR038"
+		(property "Reference" "#PWR0182"
 			(at 171.45 106.68 0)
 			(hide yes)
@@
 			(project "DDR4_DIMM"
 				(path "/2162f80d-5bbc-406a-8824-9611d78b7103/cb7293af-232b-4c7f-85bc-3b7b1ae107bd"
-					(reference "#PWR038")
+					(reference "#PWR0182")
 					(unit 1)
 				)
@@
 		(in_pos_files yes)
 		(dnp no)
-		(property "Reference" "#PWR037"
+		(property "Reference" "#PWR0181"
 			(at 124.46 85.09 0)
 			(hide yes)
@@
 			(project "DDR4_DIMM"
 				(path "/2162f80d-5bbc-406a-8824-9611d78b7103/cb7293af-232b-4c7f-85bc-3b7b1ae107bd"
-					(reference "#PWR037")
+					(reference "#PWR0181")
 					(unit 1)
 				)
@@
 		(dnp no)
 		(fields_autoplaced yes)
-		(property "Reference" "#PWR035"
+		(property "Reference" "#PWR0179"
 			(at 105.41 118.11 0)
 			(hide yes)
@@
 			(project "DDR4_DIMM"
 				(path "/2162f80d-5bbc-406a-8824-9611d78b7103/cb7293af-232b-4c7f-85bc-3b7b1ae107bd"
-					(reference "#PWR035")
+					(reference "#PWR0179")
 					(unit 1)
 				)
@@
 		(in_pos_files yes)
 		(dnp no)
-		(property "Reference" "U7"
+		(property "Reference" "U11"
 			(at 189.23 72.39 0)
 			(show_name no)
@@
 			(project "DDR4_DIMM"
 				(path "/2162f80d-5bbc-406a-8824-9611d78b7103/cb7293af-232b-4c7f-85bc-3b7b1ae107bd"
-					(reference "U7")
+					(reference "U11")
 					(unit 1)
 				)
@@
 		(in_pos_files yes)
 		(dnp no)
-		(property "Reference" "#PWR039"
+		(property "Reference" "#PWR0183"
 			(at 209.55 77.47 0)
 			(hide yes)
@@
 			(project "DDR4_DIMM"
 				(path "/2162f80d-5bbc-406a-8824-9611d78b7103/cb7293af-232b-4c7f-85bc-3b7b1ae107bd"
-					(reference "#PWR039")
-					(unit 1)
-				)
+					(reference "#PWR0183")
+					(unit 1)
+				)
