File: DDR4_DIMM.kicad_pcb (KiCad board)
At the start: 8 copper layers, 0 parts

Commit message: Adding net class, net constraint
Parts:
- added C1: 1uF, DDR4_DRAM_DIMM:C_0402_1005, F.Cu at (112.6, 101.2)
- added C10: 0.1uF, DDR4_DRAM_DIMM:C_0402_1005, F.Cu at (115.9, 103.2)
- added C11: 1uF, DDR4_DRAM_DIMM:C_0402_1005, F.Cu at (115.9, 105.2)
- added C12: 0.1uF, DDR4_DRAM_DIMM:C_0402_1005, F.Cu at (115.9, 107.1)
- added C13: 1uF, DDR4_DRAM_DIMM:C_0402_1005, F.Cu at (115.9, 109.1)
- added C14: 1uF, DDR4_DRAM_DIMM:C_0402_1005, F.Cu at (115.9, 111.1)
- added C15: 100nF, DDR4_DRAM_DIMM:C_0402_1005, F.Cu at (115.9, 113.0)
- added C16: 100nF, DDR4_DRAM_DIMM:C_0402_1005, F.Cu at (115.9, 115.0)
- added C17: 0.1uF, DDR4_DRAM_DIMM:C_0402_1005, F.Cu at (119.1, 101.2)
- added C18: 1uF, DDR4_DRAM_DIMM:C_0402_1005, F.Cu at (119.1, 103.2)
- added C19: 1uF, DDR4_DRAM_DIMM:C_0402_1005, F.Cu at (119.1, 105.2)
- added C2: 0.1uF, DDR4_DRAM_DIMM:C_0402_1005, F.Cu at (112.6, 103.2)
- added C20: 0.1uF, DDR4_DRAM_DIMM:C_0402_1005, F.Cu at (119.1, 107.1)
- added C21: 1uF, DDR4_DRAM_DIMM:C_0402_1005, F.Cu at (119.1, 109.1)
- added C22: 1uF, DDR4_DRAM_DIMM:C_0402_1005, F.Cu at (119.1, 111.1)
- added C23: 1uF, DDR4_DRAM_DIMM:C_0402_1005, F.Cu at (119.1, 113.0)
- added C24: 100nF, DDR4_DRAM_DIMM:C_0402_1005, F.Cu at (119.1, 115.0)
- added C25: 100nF, DDR4_DRAM_DIMM:C_0402_1005, F.Cu at (122.3, 101.2)
- added C26: 0.1uF, DDR4_DRAM_DIMM:C_0402_1005, F.Cu at (122.3, 103.2)
- added C27: 0.1uF, DDR4_DRAM_DIMM:C_0402_1005, F.Cu at (122.3, 105.2)
- added C28: 1uF, DDR4_DRAM_DIMM:C_0402_1005, F.Cu at (122.3, 107.1)
- added C29: 1uF, DDR4_DRAM_DIMM:C_0402_1005, F.Cu at (122.3, 109.1)
- added C3: 1uF, DDR4_DRAM_DIMM:C_0402_1005, F.Cu at (112.6, 105.2)
- added C30: 1uF, DDR4_DRAM_DIMM:C_0402_1005, F.Cu at (122.3, 111.1)
- added C31: 1uF, DDR4_DRAM_DIMM:C_0402_1005, F.Cu at (122.3, 113.0)
- added C32: 100nF, DDR4_DRAM_DIMM:C_0402_1005, F.Cu at (122.3, 115.0)
- added C33: 100nF, DDR4_DRAM_DIMM:C_0402_1005, F.Cu at (125.6, 101.2)
- added C34: 0.1uF, DDR4_DRAM_DIMM:C_0402_1005, F.Cu at (125.6, 103.2)
- added C35: 1uF, DDR4_DRAM_DIMM:C_0402_1005, F.Cu at (125.6, 105.2)
- added C36: 0.1uF, DDR4_DRAM_DIMM:C_0402_1005, F.Cu at (125.6, 107.1)
- added C37: 0.1uF, DDR4_DRAM_DIMM:C_0402_1005, F.Cu at (125.6, 109.1)
- added C38: 1uF, DDR4_DRAM_DIMM:C_0402_1005, F.Cu at (125.6, 111.1)
- added C39: 1uF, DDR4_DRAM_DIMM:C_0402_1005, F.Cu at (125.6, 113.0)
- added C4: 1uF, DDR4_DRAM_DIMM:C_0402_1005, F.Cu at (112.6, 107.1)
- added C40: 0.1uF, DDR4_DRAM_DIMM:C_0402_1005, F.Cu at (125.6, 115.0)
- added C41: 1uF, DDR4_DRAM_DIMM:C_0402_1005, F.Cu at (76.6, 101.2)
- added C42: 0.1uF, DDR4_DRAM_DIMM:C_0402_1005, F.Cu at (76.6, 103.2)
- added C43: 1uF, DDR4_DRAM_DIMM:C_0402_1005, F.Cu at (76.6, 105.2)
- added C44: 1uF, DDR4_DRAM_DIMM:C_0402_1005, F.Cu at (76.6, 107.1)
- added C45: 100nF, DDR4_DRAM_DIMM:C_0402_1005, F.Cu at (76.6, 109.1)
- added C46: 100nF, DDR4_DRAM_DIMM:C_0402_1005, F.Cu at (76.6, 111.1)
- added C47: 0.1uF, DDR4_DRAM_DIMM:C_0402_1005, F.Cu at (76.6, 113.0)
- added C48: 1uF, DDR4_DRAM_DIMM:C_0402_1005, F.Cu at (76.6, 115.0)
- added C49: 1uF, DDR4_DRAM_DIMM:C_0402_1005, F.Cu at (79.9, 101.2)
- added C5: 100nF, DDR4_DRAM_DIMM:C_0402_1005, F.Cu at (112.6, 109.1)
- added C50: 0.1uF, DDR4_DRAM_DIMM:C_0402_1005, F.Cu at (79.9, 103.2)
- added C51: 1uF, DDR4_DRAM_DIMM:C_0402_1005, F.Cu at (79.9, 105.2)
- added C52: 0.1uF, DDR4_DRAM_DIMM:C_0402_1005, F.Cu at (79.9, 107.1)
- added C53: 1uF, DDR4_DRAM_DIMM:C_0402_1005, F.Cu at (79.9, 109.1)
- added C54: 1uF, DDR4_DRAM_DIMM:C_0402_1005, F.Cu at (79.9, 111.1)
- added C55: 100nF, DDR4_DRAM_DIMM:C_0402_1005, F.Cu at (79.9, 113.0)
- added C56: 100nF, DDR4_DRAM_DIMM:C_0402_1005, F.Cu at (79.9, 115.0)
- added C57: 0.1uF, DDR4_DRAM_DIMM:C_0402_1005, F.Cu at (83.1, 101.2)
- added C58: 1uF, DDR4_DRAM_DIMM:C_0402_1005, F.Cu at (83.1, 103.2)
- added C59: 1uF, DDR4_DRAM_DIMM:C_0402_1005, F.Cu at (83.1, 105.2)
- added C6: 100nF, DDR4_DRAM_DIMM:C_0402_1005, F.Cu at (112.6, 111.1)
- added C60: 0.1uF, DDR4_DRAM_DIMM:C_0402_1005, F.Cu at (83.1, 107.1)
- added C61: 1uF, DDR4_DRAM_DIMM:C_0402_1005, F.Cu at (83.1, 109.1)
- added C62: 1uF, DDR4_DRAM_DIMM:C_0402_1005, F.Cu at (83.1, 111.1)
- added C63: 1uF, DDR4_DRAM_DIMM:C_0402_1005, F.Cu at (83.1, 113.0)
- added C64: 100nF, DDR4_DRAM_DIMM:C_0402_1005, F.Cu at (83.1, 115.0)
- added C65: 100nF, DDR4_DRAM_DIMM:C_0402_1005, F.Cu at (86.3, 101.2)
- added C66: 0.1uF, DDR4_DRAM_DIMM:C_0402_1005, F.Cu at (86.3, 103.2)
- added C67: 0.1uF, DDR4_DRAM_DIMM:C_0402_1005, F.Cu at (86.3, 105.2)
- added C68: 1uF, DDR4_DRAM_DIMM:C_0402_1005, F.Cu at (86.3, 107.1)
- added C69: 1uF, DDR4_DRAM_DIMM:C_0402_1005, F.Cu at (86.3, 109.1)
- added C7: 0.1uF, DDR4_DRAM_DIMM:C_0402_1005, F.Cu at (112.6, 113.0)
- added C70: 1uF, DDR4_DRAM_DIMM:C_0402_1005, F.Cu at (86.3, 111.1)
- added C71: 1uF, DDR4_DRAM_DIMM:C_0402_1005, F.Cu at (86.3, 113.0)
- added C72: 100nF, DDR4_DRAM_DIMM:C_0402_1005, F.Cu at (86.3, 115.0)
- added C73: 100nF, DDR4_DRAM_DIMM:C_0402_1005, F.Cu at (89.6, 101.2)
- added C74: 0.1uF, DDR4_DRAM_DIMM:C_0402_1005, F.Cu at (89.6, 103.2)
- added C75: 1uF, DDR4_DRAM_DIMM:C_0402_1005, F.Cu at (89.6, 105.2)
- added C76: 0.1uF, DDR4_DRAM_DIMM:C_0402_1005, F.Cu at (89.6, 107.1)
- added C77: 0.1uF, DDR4_DRAM_DIMM:C_0402_1005, F.Cu at (89.6, 109.1)
- added C78: 1uF, DDR4_DRAM_DIMM:C_0402_1005, F.Cu at (89.6, 111.1)
- added C79: 1uF, DDR4_DRAM_DIMM:C_0402_1005, F.Cu at (89.6, 113.0)
- added C8: 1uF, DDR4_DRAM_DIMM:C_0402_1005, F.Cu at (112.6, 115.0)
- added C80: 0.1uF, DDR4_DRAM_DIMM:C_0402_1005, F.Cu at (89.6, 115.0)
- added C81: 1uF, DDR4_DRAM_DIMM:C_0402_1005, F.Cu at (135.7, 89.1)
- added C82: 1uF, DDR4_DRAM_DIMM:C_0402_1005, F.Cu at (135.7, 91.1)
- added C83: 100nF, DDR4_DRAM_DIMM:C_0402_1005, F.Cu at (135.7, 93.1)
- added C84: 100nF, DDR4_DRAM_DIMM:C_0402_1005, F.Cu at (135.7, 95.0)
- added C85: 1nF/1005, DDR4_DRAM_DIMM:C_0402_1005, F.Cu at (135.7, 97.0)
- added C86: 10uF, DDR4_DRAM_DIMM:C_0603_1608, F.Cu at (131.9, 89.4)
- added C87: 10uF, DDR4_DRAM_DIMM:C_0603_1608, F.Cu at (131.9, 91.9)
- added C88: 10uF, DDR4_DRAM_DIMM:C_0603_1608, F.Cu at (131.9, 94.4)
- added C89: 10uF, DDR4_DRAM_DIMM:C_0603_1608, F.Cu at (131.9, 96.9)
- added C9: 1uF, DDR4_DRAM_DIMM:C_0402_1005, F.Cu at (115.9, 101.2)
- added C90: 10uF, DDR4_DRAM_DIMM:C_0603_1608, F.Cu at (131.9, 99.4)
- added C91: 1uF, DDR4_DRAM_DIMM:R_0402_1005, F.Cu at (131.3, 108.7)
- added C92: 100nF, DDR4_DRAM_DIMM:R_0402_1005, F.Cu at (131.3, 110.7)
- added CR1: SLVU2.8HTG, DDR4_DRAM_DIMM:SLVU2.8HTG, F.Cu at (140.8, 90.6)
- added D1: RCLAMP01211ZCFT, DDR4_DRAM_DIMM:RCLAMP01211ZCFT, F.Cu at (139.2, 104.7)
- added L1: MPZ1608S221A, DDR4_DRAM_DIMM:MPZ1608S260ATAH0, F.Cu at (96.1, 101.5)
- added L10: MPZ1608S221A, DDR4_DRAM_DIMM:MPZ1608S260ATAH0, F.Cu at (60.1, 104.1)
- added L11: MPZ1608S221A, DDR4_DRAM_DIMM:MPZ1608S260ATAH0, F.Cu at (60.1, 106.7)
- added L12: MPZ1608S221A, DDR4_DRAM_DIMM:MPZ1608S260ATAH0, F.Cu at (60.1, 109.3)
- added L13: MPZ1608S221A, DDR4_DRAM_DIMM:MPZ1608S260ATAH0, F.Cu at (60.1, 111.9)
- added L14: MPZ1608S221A, DDR4_DRAM_DIMM:MPZ1608S260ATAH0, F.Cu at (60.1, 114.5)
- added L15: MPZ1608S221A, DDR4_DRAM_DIMM:MPZ1608S260ATAH0, F.Cu at (60.1, 117.1)
- added L16: MPZ1608S221A, DDR4_DRAM_DIMM:MPZ1608S260ATAH0, F.Cu at (60.1, 119.7)
- added L17: MPZ1608S221A, DDR4_DRAM_DIMM:MPZ1608S260ATAH0, F.Cu at (136.5, 99.3)
- added L18: MPZ1608S221A, DDR4_DRAM_DIMM:MPZ1608S260ATAH0, F.Cu at (136.5, 101.9)
- added L19: MPZ1608S221A, DDR4_DRAM_DIMM:MPZ1608S260ATAH0, F.Cu at (135.4, 112.0)
- added L2: MPZ1608S221A, DDR4_DRAM_DIMM:MPZ1608S260ATAH0, F.Cu at (96.1, 104.1)
- added L3: MPZ1608S221A, DDR4_DRAM_DIMM:MPZ1608S260ATAH0, F.Cu at (96.1, 106.7)
- added L4: MPZ1608S221A, DDR4_DRAM_DIMM:MPZ1608S260ATAH0, F.Cu at (96.1, 109.3)
- added L5: MPZ1608S221A, DDR4_DRAM_DIMM:MPZ1608S260ATAH0, F.Cu at (96.1, 111.9)
- added L6: MPZ1608S221A, DDR4_DRAM_DIMM:MPZ1608S260ATAH0, F.Cu at (96.1, 114.5)
- added L7: MPZ1608S221A, DDR4_DRAM_DIMM:MPZ1608S260ATAH0, F.Cu at (96.1, 117.1)
- added L8: MPZ1608S221A, DDR4_DRAM_DIMM:MPZ1608S260ATAH0, F.Cu at (96.1, 119.7)
- added L9: MPZ1608S221A, DDR4_DRAM_DIMM:MPZ1608S260ATAH0, F.Cu at (60.1, 101.5)
- added R1: 15, DDR4_DRAM_DIMM:R_0402_1005, F.Cu at (99.6, 101.2)
- added R10: 15, DDR4_DRAM_DIMM:R_0402_1005, F.Cu at (102.9, 101.2)
- added R11: 15, DDR4_DRAM_DIMM:R_0402_1005, F.Cu at (102.9, 103.2)
- added R12: 15, DDR4_DRAM_DIMM:R_0402_1005, F.Cu at (102.9, 105.2)
- added R13: 15, DDR4_DRAM_DIMM:R_0402_1005, F.Cu at (102.9, 107.2)
- added R14: 15, DDR4_DRAM_DIMM:R_0402_1005, F.Cu at (102.9, 109.2)
- added R15: 15, DDR4_DRAM_DIMM:R_0402_1005, F.Cu at (102.9, 111.2)
- added R16: 15, DDR4_DRAM_DIMM:R_0402_1005, F.Cu at (102.9, 113.2)
- added R17: 15, DDR4_DRAM_DIMM:R_0402_1005, F.Cu at (102.9, 115.2)
- added R18: 240/1%, DDR4_DRAM_DIMM:R_0402_1005, F.Cu at (102.9, 117.1)
- added R19: 15, DDR4_DRAM_DIMM:R_0402_1005, F.Cu at (106.1, 101.2)
- added R2: 15, DDR4_DRAM_DIMM:R_0402_1005, F.Cu at (99.6, 103.2)
- added R20: 15, DDR4_DRAM_DIMM:R_0402_1005, F.Cu at (106.1, 103.2)
- added R21: 15, DDR4_DRAM_DIMM:R_0402_1005, F.Cu at (106.1, 105.2)
- added R22: 15, DDR4_DRAM_DIMM:R_0402_1005, F.Cu at (106.1, 107.2)
- added R23: 15, DDR4_DRAM_DIMM:R_0402_1005, F.Cu at (106.1, 109.2)
- added R24: 15, DDR4_DRAM_DIMM:R_0402_1005, F.Cu at (106.1, 111.2)
- added R25: 15, DDR4_DRAM_DIMM:R_0402_1005, F.Cu at (106.1, 113.2)
- added R26: 15, DDR4_DRAM_DIMM:R_0402_1005, F.Cu at (106.1, 115.2)
- added R27: 240/1%, DDR4_DRAM_DIMM:R_0402_1005, F.Cu at (106.1, 117.1)
- added R28: 15, DDR4_DRAM_DIMM:R_0402_1005, F.Cu at (109.4, 101.2)
- added R29: 15, DDR4_DRAM_DIMM:R_0402_1005, F.Cu at (109.4, 103.2)
- added R3: 15, DDR4_DRAM_DIMM:R_0402_1005, F.Cu at (99.6, 105.2)
- added R30: 15, DDR4_DRAM_DIMM:R_0402_1005, F.Cu at (109.4, 105.2)
- added R31: 15, DDR4_DRAM_DIMM:R_0402_1005, F.Cu at (109.4, 107.2)
- added R32: 15, DDR4_DRAM_DIMM:R_0402_1005, F.Cu at (109.4, 109.2)
- added R33: 15, DDR4_DRAM_DIMM:R_0402_1005, F.Cu at (109.4, 111.2)
- added R34: 15, DDR4_DRAM_DIMM:R_0402_1005, F.Cu at (109.4, 113.2)
- added R35: 15, DDR4_DRAM_DIMM:R_0402_1005, F.Cu at (109.4, 115.2)
- added R36: 240/1%, DDR4_DRAM_DIMM:R_0402_1005, F.Cu at (109.4, 117.1)
- added R37: 15, DDR4_DRAM_DIMM:R_0402_1005, F.Cu at (63.6, 101.2)
- added R38: 15, DDR4_DRAM_DIMM:R_0402_1005, F.Cu at (63.6, 103.2)
- added R39: 15, DDR4_DRAM_DIMM:R_0402_1005, F.Cu at (63.6, 105.2)
- added R4: 15, DDR4_DRAM_DIMM:R_0402_1005, F.Cu at (99.6, 107.2)
- added R40: 15, DDR4_DRAM_DIMM:R_0402_1005, F.Cu at (63.6, 107.2)
- added R41: 15, DDR4_DRAM_DIMM:R_0402_1005, F.Cu at (63.6, 109.2)
- added R42: 15, DDR4_DRAM_DIMM:R_0402_1005, F.Cu at (63.6, 111.2)
- added R43: 15, DDR4_DRAM_DIMM:R_0402_1005, F.Cu at (63.6, 113.2)
- added R44: 15, DDR4_DRAM_DIMM:R_0402_1005, F.Cu at (63.6, 115.2)
- added R45: 240/1%, DDR4_DRAM_DIMM:R_0402_1005, F.Cu at (63.6, 117.1)
- added R46: 15, DDR4_DRAM_DIMM:R_0402_1005, F.Cu at (66.9, 101.2)
- added R47: 15, DDR4_DRAM_DIMM:R_0402_1005, F.Cu at (66.9, 103.2)
- added R48: 15, DDR4_DRAM_DIMM:R_0402_1005, F.Cu at (66.9, 105.2)
- added R49: 15, DDR4_DRAM_DIMM:R_0402_1005, F.Cu at (66.9, 107.2)
- added R5: 15, DDR4_DRAM_DIMM:R_0402_1005, F.Cu at (99.6, 109.2)
- added R50: 15, DDR4_DRAM_DIMM:R_0402_1005, F.Cu at (66.9, 109.2)
- added R51: 15, DDR4_DRAM_DIMM:R_0402_1005, F.Cu at (66.9, 111.2)
- added R52: 15, DDR4_DRAM_DIMM:R_0402_1005, F.Cu at (66.9, 113.2)
- added R53: 15, DDR4_DRAM_DIMM:R_0402_1005, F.Cu at (66.9, 115.2)
- added R54: 240/1%, DDR4_DRAM_DIMM:R_0402_1005, F.Cu at (66.9, 117.1)
- added R55: 15, DDR4_DRAM_DIMM:R_0402_1005, F.Cu at (70.1, 101.2)
- added R56: 15, DDR4_DRAM_DIMM:R_0402_1005, F.Cu at (70.1, 103.2)
- added R57: 15, DDR4_DRAM_DIMM:R_0402_1005, F.Cu at (70.1, 105.2)
- added R58: 15, DDR4_DRAM_DIMM:R_0402_1005, F.Cu at (70.1, 107.2)
- added R59: 15, DDR4_DRAM_DIMM:R_0402_1005, F.Cu at (70.1, 109.2)
- added R6: 15, DDR4_DRAM_DIMM:R_0402_1005, F.Cu at (99.6, 111.2)
- added R60: 15, DDR4_DRAM_DIMM:R_0402_1005, F.Cu at (70.1, 111.2)
- added R61: 15, DDR4_DRAM_DIMM:R_0402_1005, F.Cu at (70.1, 113.2)
- added R62: 15, DDR4_DRAM_DIMM:R_0402_1005, F.Cu at (70.1, 115.2)
- added R63: 240/1%, DDR4_DRAM_DIMM:R_0402_1005, F.Cu at (70.1, 117.1)
- added R64: 15, DDR4_DRAM_DIMM:R_0402_1005, F.Cu at (73.4, 101.2)
- added R65: 15, DDR4_DRAM_DIMM:R_0402_1005, F.Cu at (73.4, 103.2)
- added R66: 15, DDR4_DRAM_DIMM:R_0402_1005, F.Cu at (73.4, 105.2)
- added R67: 15, DDR4_DRAM_DIMM:R_0402_1005, F.Cu at (73.4, 107.2)
- added R68: 15, DDR4_DRAM_DIMM:R_0402_1005, F.Cu at (73.4, 109.2)
- added R69: 15, DDR4_DRAM_DIMM:R_0402_1005, F.Cu at (73.4, 111.2)
- added R7: 15, DDR4_DRAM_DIMM:R_0402_1005, F.Cu at (99.6, 113.2)
- added R70: 15, DDR4_DRAM_DIMM:R_0402_1005, F.Cu at (73.4, 113.2)
- added R71: 15, DDR4_DRAM_DIMM:R_0402_1005, F.Cu at (73.4, 115.2)
- added R72: 240/1%, DDR4_DRAM_DIMM:R_0402_1005, F.Cu at (73.4, 117.1)
- added R73: 10K, DDR4_DRAM_DIMM:R_0402_1005, F.Cu at (139.9, 99.0)
- added R74: 10K, DDR4_DRAM_DIMM:R_0402_1005, F.Cu at (139.9, 101.0)
- added R75: 10K, DDR4_DRAM_DIMM:R_0402_1005, F.Cu at (139.9, 103.0)
- added R76: 10K/1%, DDR4_DRAM_DIMM:R_0603_1608, F.Cu at (131.9, 101.9)
- added R77: 10K/1%, DDR4_DRAM_DIMM:R_0603_1608, F.Cu at (131.9, 104.4)
- added R8: 15, DDR4_DRAM_DIMM:R_0402_1005, F.Cu at (99.6, 115.2)
- added R9: 240/1%, DDR4_DRAM_DIMM:R_0402_1005, F.Cu at (99.6, 117.1)
- added U1: ~, DDR4_DRAM_DIMM:DIMM_Connector_288Pin, F.Cu at (127.9, 52.9)
- added U10: TPS51200AQDRCTQ1, DDR4_DRAM_DIMM:DRC0010J, F.Cu at (139.5, 95.4)
- added U11: S-34TS04A0B-A8T5U5, DDR4_DRAM_DIMM:S-34TS04A0B-A8T5U5, F.Cu at (135.2, 109.2)
- added U2: K4A8G085WC-BCPB, DDR4_DRAM_DIMM:K4A8G085WC-BCPB, F.Cu at (97.9, 94.2)
- added U3: K4A8G085WC-BCPB, DDR4_DRAM_DIMM:K4A8G085WC-BCPB, F.Cu at (106.4, 94.2)
- added U4: K4A8G085WC-BCPB, DDR4_DRAM_DIMM:K4A8G085WC-BCPB, F.Cu at (114.9, 94.2)
- added U5: K4A8G085WC-BCPB, DDR4_DRAM_DIMM:K4A8G085WC-BCPB, F.Cu at (123.4, 94.2)
- added U6: K4A8G085WC-BCPB, DDR4_DRAM_DIMM:K4A8G085WC-BCPB, F.Cu at (61.9, 94.2)
- added U7: K4A8G085WC-BCPB, DDR4_DRAM_DIMM:K4A8G085WC-BCPB, F.Cu at (70.4, 94.2)
- added U8: K4A8G085WC-BCPB, DDR4_DRAM_DIMM:K4A8G085WC-BCPB, F.Cu at (78.9, 94.2)
- added U9: K4A8G085WC-BCPB, DDR4_DRAM_DIMM:K4A8G085WC-BCPB, F.Cu at (87.4, 94.2)
Other:
- board outline added: 133.4 x 31.8 mm
- copper layers 8 -> 6
