File: DRAM_1to4.kicad_sch (KiCad schematic)
At the start: 88 parts, among them U2 K4A8G085WC-BCPB, U3 K4A8G085WC-BCPB, U4 K4A8G085WC-BCPB, U5 K4A8G085WC-BCPB

Commit message: Adding net class, net constraint
Connections:
- net DQ32 renamed DQ0
- net DQ33 renamed DQ1
- net DQ34 renamed DQ2
- net DQ35 renamed DQ3
- net DQ36 renamed DQ4
- net DQ37 renamed DQ5
- net DQ38 renamed DQ6
- net DQ39 renamed DQ7
- net DQ40 renamed DQ8
- net DQ41 renamed DQ9
- net DQ42 renamed DQ10
- net DQ43 renamed DQ11
- net DQ44 renamed DQ12
- net DQ45 renamed DQ13
- net DQ46 renamed DQ14
- net DQ47 renamed DQ15
- net DQ48 renamed DQ16
- net DQ49 renamed DQ17
- net DQ50 renamed DQ18
- net DQ51 renamed DQ19
- net DQ52 renamed DQ20
- net DQ53 renamed DQ21
- net DQ54 renamed DQ22
- net DQ55 renamed DQ23
- net DQ56 renamed DQ24
- net DQ57 renamed DQ25
- net DQ58 renamed DQ26
- net DQ59 renamed DQ27
- net DQ60 renamed DQ28
- net DQ61 renamed DQ29
- net DQ62 renamed DQ30
- net DQ63 renamed DQ31
- net DQS4_N renamed DQS0_N
- net DQS4_P renamed DQS0_P
- net DQS5_N renamed DQS1_N
- net DQS5_P renamed DQS1_P
- net DQS6_N renamed DQS2_N
- net DQS6_P renamed DQS2_P
- net DQS7_N renamed DQS3_N
- net DQS7_P renamed DQS3_P
Changed lines of the file:
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@@
 		)
 	)
-	(global_label "DQ42"
+	(global_label "DQ10"
 		(shape bidirectional)
 		(at 121.92 124.46 180)
@@
 		)
 	)
-	(global_label "DQ56"
+	(global_label "DQ24"
 		(shape bidirectional)
 		(at 314.96 116.84 180)
@@
 		)
 	)
-	(global_label "DQS5_N"
+	(global_label "DQS1_N"
 		(shape input)
 		(at 138.43 151.13 180)
@@
 		)
 	)
-	(global_label "DQ49"
+	(global_label "DQ17"
 		(shape bidirectional)
 		(at 214.63 120.65 180)
@@
 		)
 	)
-	(global_label "DQS7_N"
+	(global_label "DQS3_N"
 		(shape input)
 		(at 331.47 151.13 180)
@@
 		)
 	)
-	(global_label "DQ59"
+	(global_label "DQ27"
 		(shape bidirectional)
 		(at 314.96 128.27 180)
@@
 		)
 	)
-	(global_label "DQ55"
+	(global_label "DQ23"
 		(shape bidirectional)
 		(at 214.63 143.51 180)
@@
 		)
 	)
-	(global_label "DQS7_P"
+	(global_label "DQS3_P"
 		(shape input)
 		(at 331.47 147.32 180)
@@
 		)
 	)
-	(global_label "DQ40"
+	(global_label "DQ8"
 		(shape bidirectional)
 		(at 121.92 116.84 180)
@@
 		)
 		(property "Intersheetrefs" "${INTERSHEET_REFS}"
-			(at 112.804 116.84 0)
+			(at 114.0135 116.84 0)
 			(hide yes)
 			(show_name no)
@@
 		)
 	)
-	(global_label "DQS6_N"
+	(global_label "DQS2_N"
 		(shape input)
 		(at 231.14 151.13 180)
@@
 		)
 	)
-	(global_label "DQ44"
+	(global_label "DQ12"
 		(shape bidirectional)
 		(at 121.92 132.08 180)
@@
 		)
 	)
-	(global_label "DQ61"
+	(global_label "DQ29"
 		(shape bidirectional)
 		(at 314.96 135.89 180)
@@
 		)
 	)
-	(global_label "DQ62"
+	(global_label "DQ30"
 		(shape bidirectional)
 		(at 314.96 139.7 180)
@@
 		)
 	)
-	(global_label "DQ32"
+	(global_label "DQ0"
 		(shape bidirectional)
 		(at 31.75 116.84 180)
@@
 		)
 		(property "Intersheetrefs" "${INTERSHEET_REFS}"
-			(at 22.634 116.84 0)
+			(at 23.8435 116.84 0)
 			(hide yes)
 			(show_name no)
@@
 		)
 	)
-	(global_label "DQ43"
+	(global_label "DQ11"
 		(shape bidirectional)
 		(at 121.92 128.27 180)
@@
 		)
 	)
-	(global_label "DQS5_P"
+	(global_label "DQS1_P"
 		(shape input)
 		(at 138.43 147.32 180)
@@
 		)
 	)
-	(global_label "DQS4_N"
+	(global_label "DQS0_N"
 		(shape input)
 		(at 48.26 151.13 180)
@@
 		)
 	)
-	(global_label "DQ37"
+	(global_label "DQ5"
 		(shape bidirectional)
 		(at 31.75 135.89 180)
@@
 		)
 		(property "Intersheetrefs" "${INTERSHEET_REFS}"
-			(at 22.634 135.89 0)
+			(at 23.8435 135.89 0)
 			(hide yes)
 			(show_name no)
@@
 		)
 	)
-	(global_label "DQ63"
+	(global_label "DQ31"
 		(shape bidirectional)
 		(at 314.96 143.51 180)
@@
 		)
 	)
-	(global_label "DQ47"
+	(global_label "DQ15"
 		(shape bidirectional)
 		(at 121.92 143.51 180)
@@
 		)
 	)
-	(global_label "DQS6_P"
+	(global_label "DQS2_P"
 		(shape input)
 		(at 231.14 147.32 180)
@@
 		)
 	)
-	(global_label "DQ35"
+	(global_label "DQ3"
 		(shape bidirectional)
 		(at 31.75 128.27 180)
@@
 		)
 		(property "Intersheetrefs" "${INTERSHEET_REFS}"
-			(at 22.634 128.27 0)
+			(at 23.8435 128.27 0)
 			(hide yes)
 			(show_name no)
@@
 		)
 	)
-	(global_label "DQ58"
+	(global_label "DQ26"
 		(shape bidirectional)
 		(at 314.96 124.46 180)
@@
 		)
 	)
-	(global_label "DQ57"
+	(global_label "DQ25"
 		(shape bidirectional)
 		(at 314.96 120.65 180)
@@
 		)
 	)
-	(global_label "DQ52"
+	(global_label "DQ20"
 		(shape bidirectional)
 		(at 214.63 132.08 180)
@@
 		)
 	)
-	(global_label "DQ48"
+	(global_label "DQ16"
 		(shape bidirectional)
 		(at 214.63 116.84 180)
@@
 		)
 	)
-	(global_label "DQ53"
+	(global_label "DQ21"
 		(shape bidirectional)
 		(at 214.63 135.89 180)
@@
 		)
 	)
-	(global_label "DQ36"
+	(global_label "DQ4"
 		(shape bidirectional)
 		(at 31.75 132.08 180)
@@
 		)
 		(property "Intersheetrefs" "${INTERSHEET_REFS}"
-			(at 22.634 132.08 0)
+			(at 23.8435 132.08 0)
 			(hide yes)
 			(show_name no)
@@
 		)
 	)
-	(global_label "DQ33"
+	(global_label "DQ1"
 		(shape bidirectional)
 		(at 31.75 120.65 180)
@@
 		)
 		(property "Intersheetrefs" "${INTERSHEET_REFS}"
-			(at 22.634 120.65 0)
+			(at 23.8435 120.65 0)
 			(hide yes)
 			(show_name no)
@@
 		)
 	)
-	(global_label "DQ50"
+	(global_label "DQ18"
 		(shape bidirectional)
 		(at 214.63 124.46 180)
@@
 		)
 	)
-	(global_label "DQ41"
+	(global_label "DQ9"
 		(shape bidirectional)
 		(at 121.92 120.65 180)
@@
 		)
 		(property "Intersheetrefs" "${INTERSHEET_REFS}"
-			(at 112.804 120.65 0)
+			(at 114.0135 120.65 0)
 			(hide yes)
 			(show_name no)
@@
 		)
 	)
-	(global_label "DQ46"
+	(global_label "DQ14"
 		(shape bidirectional)
 		(at 121.92 139.7 180)
@@
 		)
 	)
-	(global_label "DQ38"
+	(global_label "DQ6"
 		(shape bidirectional)
 		(at 31.75 139.7 180)
@@
 		)
 		(property "Intersheetrefs" "${INTERSHEET_REFS}"
-			(at 22.634 139.7 0)
+			(at 23.8435 139.7 0)
 			(hide yes)
 			(show_name no)
@@
 		)
 	)
-	(global_label "DQ51"
+	(global_label "DQ19"
 		(shape bidirectional)
 		(at 214.63 128.27 180)
@@
 		)
 	)
-	(global_label "DQ54"
+	(global_label "DQ22"
 		(shape bidirectional)
 		(at 214.63 139.7 180)
@@
 		)
 	)
-	(global_label "DQ39"
+	(global_label "DQ7"
 		(shape bidirectional)
 		(at 31.75 143.51 180)
@@
 		)
 		(property "Intersheetrefs" "${INTERSHEET_REFS}"
-			(at 22.634 143.51 0)
+			(at 23.8435 143.51 0)
 			(hide yes)
 			(show_name no)
@@
 		)
 	)
-	(global_label "DQ45"
+	(global_label "DQ13"
 		(shape bidirectional)
 		(at 121.92 135.89 180)
@@
 		)
 	)
-	(global_label "DQ60"
+	(global_label "DQ28"
 		(shape bidirectional)
 		(at 314.96 132.08 180)
@@
 		)
 	)
-	(global_label "DQ34"
+	(global_label "DQ2"
 		(shape bidirectional)
 		(at 31.75 124.46 180)
@@
 		)
 		(property "Intersheetrefs" "${INTERSHEET_REFS}"
-			(at 22.634 124.46 0)
+			(at 23.8435 124.46 0)
 			(hide yes)
 			(show_name no)
@@
 		)
 	)
-	(global_label "DQS4_P"
+	(global_label "DQS0_P"
 		(shape input)
 		(at 48.26 147.32 180)
